File: KiCad/TrackerFrontPanel/pwr.sch (KiCad schematic (older format))
At the start: 10 parts, among them U1 STM32F303V(B-C)Tx_u

Commit message: save prior to updating to kicad 5
Changed lines of the file:
@@
 F 0 "U1" H 2150 3800 50  0000 C CNN
 F 1 "STM32F303V(B-C)Tx_u" H 2150 3650 50  0000 C CNN
-F 2 "Housings_QFP:LQFP-100_14x14mm_Pitch0.5mm" H 2050 3500 50  0000 C CIN
+F 2 "Housings_QFP:LQFP-100_14x14mm_Pitch0.5mm" H 2050 3500 50  0001 C CIN
 F 3 "" H 3050 3600 50  0000 C CNN
 	8    3050 3600
@@
 F 0 "U1" H 2250 2100 50  0000 C CNN
 F 1 "STM32F303V(B-C)Tx_u" H 2350 2000 50  0000 C CNN
-F 2 "Housings_QFP:LQFP-100_14x14mm_Pitch0.5mm" H 2250 1850 50  0000 C CIN
+F 2 "Housings_QFP:LQFP-100_14x14mm_Pitch0.5mm" H 2250 1850 50  0001 C CIN
 F 3 "" H 3050 2100 50  0000 C CNN
 	9    3050 2100
@@
 F 0 "U1" H 2750 1150 50  0000 C CNN
 F 1 "STM32F303V(B-C)Tx_u" H 2650 1000 50  0000 C CNN
-F 2 "Housings_QFP:LQFP-100_14x14mm_Pitch0.5mm" H 2700 850 50  0000 C CIN
+F 2 "Housings_QFP:LQFP-100_14x14mm_Pitch0.5mm" H 2700 850 50  0001 C CIN
 F 3 "" H 3400 1050 50  0000 C CNN
 	7    3400 1050
