File: KiCad/TrackerFrontPanel/sw-led.sch (KiCad schematic (older format))
At the start: 19 parts, among them SW1 SW_SPST, SW10 SW_SPST, SW2 SW_SPST, SW3 SW_SPST, SW4 SW_SPST, SW5 SW_SPST, SW6 SW_SPST, SW7 SW_SPST, SW8 SW_SPST, SW9 SW_SPST, U1 STM32F303V(B-C)Tx_u

Commit message: save prior to updating to kicad 5
Parts:
- removed SW1, SW10, SW2, SW3, SW4, SW5, SW6, SW7, SW8, SW9: SW_SPST, symbol SW_SPST
- added SW1, SW10, SW2, SW3, SW4, SW5, SW6, SW7, SW8, SW9: TS001, footprints:PTS125, symbol TS001
- D1, D2, D3, D4: footprint (none) -> Diodes_SMD:D_1206
- R1, R2, R3, R4: footprint (none) -> Resistors_SMD:R_1206
- U1: footprint LQFP100 -> Housings_QFP:LQFP-100_14x14mm_Pitch0.5mm
Connections:
- net GND: now also SW1.3 (B1), SW1.4 (B2), SW10.4 (B2), SW2.3 (B1), SW2.4 (B2), SW3.3 (B1), SW3.4 (B2), SW4.3 (B1), SW4.4 (B2), SW5.3 (B1), SW5.4 (B2), SW6.3 (B1), SW6.4 (B2), SW7.3 (B1), SW7.4 (B2), SW8.3 (B1), SW8.4 (B2), SW9.3 (B1), SW9.4 (B2)
- net at U1.15 (PC0/ADC1_IN6/ADC2_IN6/COMP7_INM): now also SW10.1 (A1), SW10.2 (A2)
- net at U1.16 (PC1/ADC1_IN7/ADC2_IN7/COMP7_INP): now also SW9.1 (A1), SW9.2 (A2)
- net at U1.17 (PC2/ADC1_IN8/ADC2_IN8/ADC3_EXTI2/ADC4_EXTI2/COMP7_OUT): now also SW8.1 (A1), SW8.2 (A2)
- net at U1.18 (PC3/ADC1_IN9/ADC2_IN9/TIM1_BKIN2): now also SW7.1 (A1), SW7.2 (A2)
- net at U1.33 (PC4/ADC2_IN5/USART1_TX): now also SW6.1 (A1), SW6.2 (A2)
- net at U1.34 (PC5/ADC2_IN11/OPAMP1_VINM/OPAMP1_VINM_SEC/OPAMP2_VINM/OPAMP2_VINM_SEC/TSC_G3_IO1/USART1_RX): now also SW5.1 (A1), SW5.2 (A2)
- net at U1.63 (PC6/COMP6_OUT/I2S2_MCK/TIM3_CH1/TIM8_CH1): now also SW4.1 (A1), SW4.2 (A2)
- net at U1.64 (PC7/COMP5_OUT/I2S3_MCK/TIM3_CH2/TIM8_CH2): now also SW3.1 (A1), SW3.2 (A2)
- net at U1.65 (PC8/COMP3_OUT/TIM3_CH3/TIM8_CH3): now also SW2.1 (A1), SW2.2 (A2)
- net at U1.66 (PC9/DAC_EXTI9/I2S_CKIN/TIM3_CH4/TIM8_BKIN2/TIM8_CH4): now also SW1.1 (A1), SW1.2 (A2)
