File: KiCad/TrackerFrontPanel/_saved_FrontPanel.sch (KiCad schematic (older format))
At the start: 5 parts, among them J1 Conn_01x08, J2 Conn_01x20, J3 Conn_02x04_Odd_Even, J4 Conn_01x06, U1 STM32F303V(B-C)Tx_u

Commit message: get ready to transfer back to main computer
Parts:
- J1: symbol Conn_01x08 -> FrontPanel-rescue:Conn_01x08
- J2: symbol Conn_01x20 -> FrontPanel-rescue:Conn_01x20
- J3: symbol Conn_02x04_Odd_Even -> FrontPanel-rescue:Conn_02x04_Odd_Even
- J4: symbol Conn_01x06 -> FrontPanel-rescue:Conn_01x06
- U1: symbol STM32F303V(B-C)Tx_u -> stm32:STM32F303V(B-C)Tx_u
Connections:
- net ~RST: now reaches J2.16 (Pin_16), U1.51 (PB12/ADC4_IN3/COMP3_INM/I2C2_SMBA/I2S2_WS/OPAMP4_VOUT/SPI2_NSS/TIM1_BKIN/TSC_G6_IO2/USART3_CK)
- net ~CS: now reaches J2.17 (Pin_17), U1.96 (PB9/CAN_TX/COMP2_OUT/DAC_EXTI9/I2C1_SDA/IR_OUT/TIM17_CH1/TIM4_CH4/TIM8_CH3)
- net D\~C: now reaches J2.4 (Pin_4), U1.47 (PB10/COMP5_INM/OPAMP3_VINM/OPAMP3_VINM_SEC/OPAMP4_VINM/OPAMP4_VINM_SEC/TIM2_CH3/TSC_SYNC/USART3_TX)
- net CLK: now reaches J2.7 (Pin_7), U1.52 (PB13/ADC3_IN5/COMP5_INP/I2S2_CK/OPAMP3_VINP/OPAMP3_VINP_SEC/OPAMP4_VINP/OPAMP4_VINP_SEC/SPI2_SCK/TIM1_CH1N/TSC_G6_IO3/USART3_CTS)
- net MOSI: now reaches J2.8 (Pin_8), U1.54 (PB15/ADC1_EXTI15/ADC2_EXTI15/ADC4_IN5/COMP6_INM/I2S2_SD/RTC_REFIN/SPI2_MOSI/TIM15_CH1N/TIM15_CH2/TIM1_CH3N)
Changed lines of the file:
@@
-EESchema Schematic File Version 2
-LIBS:power
-LIBS:device
-LIBS:switches
-LIBS:relays
-LIBS:motors
-LIBS:transistors
-LIBS:conn
-LIBS:linear
-LIBS:regul
-LIBS:74xx
-LIBS:cmos4000
-LIBS:adc-dac
-LIBS:memory
-LIBS:xilinx
-LIBS:microcontrollers
-LIBS:dsp
-LIBS:microchip
-LIBS:analog_switches
-LIBS:motorola
-LIBS:texas
-LIBS:intel
-LIBS:audio
-LIBS:interface
-LIBS:digital-audio
-LIBS:philips
-LIBS:display
-LIBS:cypress
-LIBS:siliconi
-LIBS:opto
-LIBS:atmel
-LIBS:contrib
-LIBS:valves
-LIBS:stm32
-LIBS:MyParts
+EESchema Schematic File Version 4
 LIBS:FrontPanel-cache
-EELAYER 25 0
+EELAYER 26 0
 EELAYER END
 $Descr A4 11693 8268
@@
 $EndDescr
 $Comp
-L Conn_01x20 J2
+L FrontPanel-rescue:Conn_01x20 J2
 U 1 1 5B96B692
 P 2700 5100
@@
 $EndComp
 $Comp
-L Conn_01x06 J4
+L FrontPanel-rescue:Conn_01x06 J4
 U 1 1 5B96B7B2
 P 5200 7300
@@
 $EndComp
 $Comp
-L Conn_02x04_Odd_Even J3
+L FrontPanel-rescue:Conn_02x04_Odd_Even J3
 U 1 1 5B96B85D
 P 3700 1000
@@
 $EndComp
 $Comp
-L GND #PWR01
+L power:GND #PWR01
 U 1 1 5B96B92C
 P 4200 900
@@
 $EndComp
 $Comp
-L +3.3V #PWR02
+L power:+3.3V #PWR02
 U 1 1 5B96B94A
 P 4200 1000
@@
 $EndComp
 $Comp
-L GND #PWR03
+L power:GND #PWR03
 U 1 1 5B96BA03
 P 5400 6900
@@
 NoConn ~ 4900 7100
 $Comp
-L GND #PWR04
+L power:GND #PWR04
 U 1 1 5B96BB70
 P 3100 6000
@@
 $EndComp
 $Comp
-L +3.3V #PWR05
+L power:+3.3V #PWR05
 U 1 1 5B96BB8E
 P 3100 5900
@@
 NoConn ~ 2900 5800
 $Comp
-L GND #PWR06
+L power:GND #PWR06
 U 1 1 5B96BC1B
 P 3100 4100
@@
 TX
 $Comp
-L Conn_01x08 J1
+L FrontPanel-rescue:Conn_01x08 J1
 U 1 1 5B96C9E9
 P 1200 2200
@@
 NB: use only Straight through Ethernet cable-
 $Comp
-L GND #PWR07
+L power:GND #PWR07
 U 1 1 5B96CC13
 P 1600 1850
@@
 $EndComp
 $Comp
-L +3.3V #PWR08
+L power:+3.3V #PWR08
 U 1 1 5B96CC33
 P 1600 2450
@@
 	1400 1800 1600 1800
 Wire Wire Line
-	1600 1800 1600 1900
+	1600 1800 1600 1850
 Wire Wire Line
 	1600 1900 1400 1900
@@
 	1400 2400 1600 2400
 Wire Wire Line
-	1600 2400 1600 2500
+	1600 2400 1600 2450
 Wire Wire Line
 	1600 2500 1400 2500
@@
 $EndSheet
 $Comp
-L STM32F303V(B-C)Tx_u U1
+L stm32:STM32F303V(B-C)Tx_u U1
 U 1 1 5B96D604
 P 11400 1600
@@
 $EndComp
 $Comp
-L STM32F303V(B-C)Tx_u U1
+L stm32:STM32F303V(B-C)Tx_u U1
 U 2 1 5B96D829
 P 9500 4900
@@
 NoConn ~ 4000 1100
 NoConn ~ 4000 1200
+Wire Wire Line
+	1600 1850 1600 1900
+Wire Wire Line
+	1600 2450 1600 2500
+Text Label 3350 5700 0    50   ~ 0
+D\~C
+Text Label 3300 5400 0    50   ~ 0
+CLK
+Text Label 3550 5300 0    50   ~ 0
+MOSI
+Text Label 3450 4500 0    50   ~ 0
+~RST
+Text Label 3250 4400 0    50   ~ 0
+~CS
 $EndSCHEMATC
