File: KiCad/TrackerBackPanel/C-D.sch (KiCad schematic (older format))
At the start: 8 parts, among them J4 Conn_01x02, J5 Conn_01x02, J6 Conn_01x02, J7 Conn_01x02, J8 Conn_01x04, J9 Conn_01x04, SW1 SW-DIP-8, U1 STM32F303V(B-C)Tx_u

Commit message: update circuit board with new changes;
Parts:
- SW1: footprint Button_Switch_SMD:SW_DIP_SPSTx08_Slide_6.7x21.88mm_W6.73mm_P2.54mm_LowProfile_JPin -> Button_Switch_SMD:SW_DIP_SPSTx08_Slide_6.7x21.88mm_W8.61mm_P2.54mm_LowProfile
Other:
- note added: "NB - These have been switched on purpose -\nindustry is labelled opposite of what the chip says.\n\n"
Changed lines of the file:
@@
 $EndComp
-Wire Wire Line
-	950  750  950  800
-Wire Wire Line
-	950  1200 950  1250
 Wire Wire Line
 	950  1550 950  1600
@@
 	950  1900 950  2000
 Wire Wire Line
-	1450 2000 1450 800
-Wire Wire Line
-	1450 800  950  800
-Wire Wire Line
 	1450 2000 2100 2000
-Connection ~ 950  800
-Wire Wire Line
-	950  800  950  850
-Wire Wire Line
-	950  1250 1700 1250
-Wire Wire Line
-	1700 1250 1700 1850
 Wire Wire Line
 	1700 1850 2100 1850
-Connection ~ 950  1250
-Wire Wire Line
-	950  1250 950  1300
 $Comp
 L power:GND #PWR013
@@
 Wire Wire Line
 	950  1600 950  1650
-Text Label 1150 800  0    50   ~ 0
-RS485A(-)
-Text Label 1100 1250 0    50   ~ 0
-RS485B(+)
 Text Label 1050 1600 0    50   ~ 0
 RS485C
@@
 F 0 "SW1" H 4600 3813 60  0000 C CNN
 F 1 "SW-DIP-8" H 4600 3919 60  0000 C CNN
-F 2 "Button_Switch_SMD:SW_DIP_SPSTx08_Slide_6.7x21.88mm_W6.73mm_P2.54mm_LowProfile_JPin" H 4600 4550 60  0001 C CNN
+F 2 "Button_Switch_SMD:SW_DIP_SPSTx08_Slide_6.7x21.88mm_W8.61mm_P2.54mm_LowProfile" H 4600 4550 60  0001 C CNN
 F 3 "" H 4600 4550 60  0000 C CNN
 	1    4600 4550
@@
 Wire Wire Line
 	3900 4550 3900 4700
+Wire Wire Line
+	950  1200 950  1250
+Wire Wire Line
+	950  750  950  800
+Wire Wire Line
+	1450 2000 1450 1250
+Wire Wire Line
+	1450 1250 950  1250
+Connection ~ 950  1250
+Wire Wire Line
+	950  1250 950  1300
+Wire Wire Line
+	1700 800  950  800
+Wire Wire Line
+	1700 800  1700 1850
+Connection ~ 950  800
+Wire Wire Line
+	950  800  950  850
+Text Label 1200 800  0    50   ~ 0
+RS485A(-)
+Text Label 1150 1250 0    50   ~ 0
+RS485B(+)
+Text Notes 2100 850  0    50   ~ 0
+NB - These have been switched on purpose -\nindustry is labelled opposite of what the chip says.\n\n
 $EndSCHEMATC
