File: KiCad/TrackerBackPanel/serial.sch (KiCad schematic (older format))
At the start: 18 parts, among them U3 SN65HV7X, U4 SN65HV7X

Commit message: update circuit board with new changes;
Parts:
- R1, R2, R3, R4: footprint Resistor_SMD:R_1812_4532Metric -> Resistor_SMD:R_2816_7142Metric_Pad3.20x4.45mm_HandSolder
Changed lines of the file:
@@
 F 0 "R3" V 7130 1100 50  0000 C CNN
 F 1 "10" V 7050 1100 50  0000 C CNN
-F 2 "Resistor_SMD:R_1812_4532Metric" V 6980 1100 50  0001 C CNN
+F 2 "Resistor_SMD:R_2816_7142Metric_Pad3.20x4.45mm_HandSolder" V 6980 1100 50  0001 C CNN
 F 3 "" H 7050 1100 50  0001 C CNN
 	1    7050 1100
@@
 F 0 "R4" V 7130 1800 50  0000 C CNN
 F 1 "10" V 7050 1800 50  0000 C CNN
-F 2 "Resistor_SMD:R_1812_4532Metric" V 6980 1800 50  0001 C CNN
+F 2 "Resistor_SMD:R_2816_7142Metric_Pad3.20x4.45mm_HandSolder" V 6980 1800 50  0001 C CNN
 F 3 "" H 7050 1800 50  0001 C CNN
 	1    7050 1800
@@
 F 0 "R1" V 7030 4650 50  0000 C CNN
 F 1 "10" V 6950 4650 50  0000 C CNN
-F 2 "Resistor_SMD:R_1812_4532Metric" V 6880 4650 50  0001 C CNN
+F 2 "Resistor_SMD:R_2816_7142Metric_Pad3.20x4.45mm_HandSolder" V 6880 4650 50  0001 C CNN
 F 3 "" H 6950 4650 50  0001 C CNN
 	1    6950 4650
@@
 F 0 "R2" V 7030 5350 50  0000 C CNN
 F 1 "10" V 6950 5350 50  0000 C CNN
-F 2 "Resistor_SMD:R_1812_4532Metric" V 6880 5350 50  0001 C CNN
+F 2 "Resistor_SMD:R_2816_7142Metric_Pad3.20x4.45mm_HandSolder" V 6880 5350 50  0001 C CNN
 F 3 "" H 6950 5350 50  0001 C CNN
 	1    6950 5350
