File: KiCad/TrackerBackPanel/BackPanel.kicad_pcb (KiCad board)
At the start: 2 copper layers, 112 x 125.1 mm, 45 parts, among them J1 Conn_01x08, J10 Conn_01x03, J2 Conn_02x04_Odd_Even, J3 Conn_01x06, J4 Conn_01x02, J5 Conn_01x02, J6 Conn_01x02, J7 Conn_01x02, J8 Conn_01x04, J9 Conn_01x04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

Commit message: update circuit board with new changes;
Parts:
- added C12: 220uF, Capacitor_SMD:CP_Elec_10x10, F.Cu at (113.4, 73.8)
- added C13: 100uF, Capacitor_SMD:CP_Elec_6.3x5.2, F.Cu at (174.0, 112.8)
- added C14: 1uF, Capacitor_SMD:C_1206_3216Metric, F.Cu at (177.8, 144.5)
- added C15: 1uF, Capacitor_SMD:C_1206_3216Metric, F.Cu at (172.7, 144.4)
- added C16: 100uF, Capacitor_SMD:CP_Elec_6.3x5.2, F.Cu at (184.9, 112.8)
- added J11: Conn_01x02, TerminalBlock:TerminalBlock_Altech_AK300-2_P5.00mm, F.Cu at (184.8, 34.3)
- C8: value 100uF -> 220uF; footprint Capacitor_SMD:CP_Elec_5x5.3 -> Capacitor_SMD:CP_Elec_10x10
- R1, R2, R3, R4: footprint Resistor_SMD:R_1812_4532Metric -> Resistor_SMD:R_2816_7142Metric_Pad3.20x4.45mm_HandSolder
- SW1: footprint Button_Switch_SMD:SW_DIP_SPSTx08_Slide_6.7x21.88mm_W6.73mm_P2.54mm_LowProfile_JPin -> Button_Switch_SMD:SW_DIP_SPSTx08_Slide_6.7x21.88mm_W8.61mm_P2.54mm_LowProfile
- moved J3 31.2 mm to (163.8, 59.4), turned to 180 degrees
- moved C8 25.9 mm to (125.5, 73.7), turned to 270 degrees
- moved R2 3.63 mm to (142.0, 94.4), turned to 90 degrees
- moved R4 3.12 mm to (111.7, 111.0), turned to 0 degrees
- moved R3 2.97 mm to (124.2, 110.7), turned to 180 degrees
- moved SW1 1.21 mm to (152.0, 33.5), turned to 270 degrees
- moved R1 0.62 mm to (142.0, 83.1), turned to 90 degrees
Connections:
- F3 pad 1: /C-D/RS485B(+) -> /C-D/RS485A(-)
- F4 pad 1: /C-D/RS485A(-) -> /C-D/RS485B(+)
- RV3 pad 1: /C-D/RS485B(+) -> /C-D/RS485A(-)
- RV4 pad 1: /C-D/RS485A(-) -> /C-D/RS485B(+)
- U1 pad 38: /GPIOE/GoWest -> /GPIOE/CurrentSense
- U1 pad 40: Net-(U1-Pad40) -> /GPIOE/pwm
- U1 pad 5: /GPIOE/CurrentSense -> /GPIOE/GoWest
- U5 pad 1: /GPIOE/CurrentSense -> /GPIOE/GoWest
- U5 pad 3: +3V3 -> /GPIOE/pwm
- U5 pad 4: /GPIOE/GoWest -> /GPIOE/CurrentSense
Routing:
- net GND: track 583.5 -> 663.1 mm, vias 1 -> 0
- net +24V: track 130.0 -> 190.0 mm
- net /GPIOE/EastLimit: track 108.1 -> 164.6 mm, vias 0 -> 1
- net /GPIOE/pwm: track 0.00 -> 52.7 mm
- net /GPIOE/CurrentSense: track 87.9 -> 51.4 mm
- net +3V3: track 294.2 -> 259.0 mm
- net Net-(J3-Pad5): track 54.3 -> 26.8 mm, vias 1 -> 0
- net Net-(J3-Pad4): track 51.0 -> 27.1 mm, vias 1 -> 0
- net /GPIOE/WestLimit: track 101.7 -> 125.5 mm
- net /C-D/serial/TX_en: track 80.8 -> 58.7 mm, vias 0 -> 2
- net /C-D/serial/RX: track 76.2 -> 54.3 mm, vias 0 -> 2
- net Net-(SW1-Pad7): track 41.6 -> 21.6 mm
- net /GPIOE/GoWest: track 50.5 -> 68.0 mm
- net /C-D/RS485B(+): track 63.4 -> 46.2 mm
- net Net-(J2-Pad1): track 48.4 -> 31.9 mm, vias 0 -> 1
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Other:
- board text added: "RS485A(-)"
- board text added: "RS485B(+)"
- board text removed: "RS485A"
- board text removed: "RS485B"

Commit message: Add all files and check in prior to mothballing
Parts:
- C10, C11: value .1u -> .1uF
- R1, R2, R3, R4: value 10 -> TBU; footprint Resistor_SMD:R_2816_7142Metric_Pad3.20x4.45mm_HandSolder -> CH20M:TBU
- moved R2 0.44 mm to (142.0, 94.0), turned to 270 degrees
- moved R1 0.40 mm to (142.3, 83.3), turned to 270 degrees
- moved R3 0.36 mm to (123.9, 110.6), turned to 0 degrees
- moved R4 0.34 mm to (112.0, 110.8), turned to 180 degrees
Connections:
- C15 pad 1: /GPIOE/WestLimit -> /GPIOE/GoWest
- C16 pad 1: /GPIOE/WestLimit -> /GPIOE/GoWest
- J10 pad 2: /GPIOE/WestLimit -> /GPIOE/GoWest
- U1 pad 2: /GPIOE/WestLimit -> /GPIOE/GoWest
- U1 pad 4: /GPIOE/GoEast -> /GPIOE/EastLimit
- U5 pad 6: /GPIOE/GoEast -> /GPIOE/EastLimit
Routing:
- net /GPIOE/GoWest: track 68.0 -> 218.1 mm
- net /GPIOE/WestLimit: track 125.5 -> 0.00 mm
- net /GPIOE/EastLimit: track 164.6 -> 256.9 mm, vias 1 -> 2
- net /GPIOE/GoEast: track 68.5 -> 0.00 mm, vias 1 -> 0
- net GND: track 663.1 -> 657.7 mm
